Commit message: Fix various files

File: robot_arm/urdf/robot_arm.urdf (robot description, URDF)
Before this commit: robot robot_arm, 5 links, 4 joints
Links:
- removed link Gripper
- added link Gripper_1, mass 0.00733041741689851; collision mesh filename=package://robot_arm/meshes/Gripper_1.STL; visual mesh filename=package://robot_arm/meshes/Gripper_1.STL
- added link Gripper_2, mass 0.00782008836001168; collision mesh filename=package://robot_arm/meshes/Gripper_2.STL; visual mesh filename=package://robot_arm/meshes/Gripper_2.STL
- link Link_1: mass 0.14143 -> 0.14588
- link Link_3: mass 0.01296 -> 0.0129599236993002
- link Link_4: mass 0.022295 -> 0.022474
Joints:
- added joint Joint_5: type revolute, parent Link_4, child Gripper_2, origin xyz=-0.009 0 0.075 rpy=0 0 0, axis 0 1 0, limit lower=-1.6 upper=1.6 effort=200 velocity=1.0
- joint Joint_1: axis 0 0 0 -> 0 0 -1; origin xyz=0 0 0.07 rpy=0 0 0 -> xyz=0 0 0.06 rpy=0 0 0
- joint Joint_2: axis 0 -1 0 -> 0 1 0; origin xyz=0 0 0.042 rpy=0 0 0 -> xyz=0 0 0.052 rpy=0 0 0
- joint Joint_4: child Gripper -> Gripper_1

File: robot_arm/urdf/robot_arm_control.urdf (robot description, URDF)
Before this commit: robot robot_arm, 5 links, 4 joints
Links:
- removed link Gripper
- added link Gripper_1, mass 0.00733041741689851; collision mesh filename=package://robot_arm/meshes/Gripper_1.STL scale=1 1 1; visual mesh filename=package://robot_arm/meshes/Gripper_1.STL scale=1 1 1
- added link Gripper_2, mass 0.00782008836001168; collision mesh filename=package://robot_arm/meshes/Gripper_2.STL scale=1 1 1; visual mesh filename=package://robot_arm/meshes/Gripper_2.STL scale=1 1 1
- link Link_1: mass 0.14143 -> 5.4588; geometry collision mesh filename=package://robot_arm/meshes/Link_1.STL scale=1 1 1; visual mesh filename=package://robot_arm/meshes/Link_1.STL scale=1 1 1
- link Link_2: geometry collision mesh filename=package://robot_arm/meshes/Link_2.STL scale=1 1 1; visual mesh filename=package://robot_arm/meshes/Link_2.STL scale=1 1 1
- link Link_3: mass 0.01296 -> 0.0129599236993002; geometry collision mesh filename=package://robot_arm/meshes/Link_3.STL scale=1 1 1; visual mesh filename=package://robot_arm/meshes/Link_3.STL scale=1 1 1
- link Link_4: mass 0.022295 -> 0.022474; geometry collision mesh filename=package://robot_arm/meshes/Link_4.STL scale=1 1 1; visual mesh filename=package://robot_arm/meshes/Link_4.STL scale=1 1 1
Joints:
- added joint Joint_5: type revolute, parent Link_4, child Gripper_2, origin xyz=-0.009 0 0.075 rpy=0 0 0, axis 0 1 0, limit lower=-0.4 upper=0.4 effort=2.0 velocity=0.5
- joint Joint_1: axis 0 0 0 -> 0 0 -1; limit lower=-1.6 upper=1.6 effort=200 velocity=1.0 -> lower=-1.6 upper=1.6 effort=200 velocity=0.1; origin xyz=0 0 0.07 rpy=0 0 0 -> xyz=0 0 0.06 rpy=0 0 0
- joint Joint_2: axis 0 -1 0 -> 0 1 0; limit lower=-1.6 upper=1.6 effort=200 velocity=1.0 -> lower=-1.6 upper=1.6 effort=200 velocity=0.1; origin xyz=0 0 0.042 rpy=0 0 0 -> xyz=0 0 0.052 rpy=0 0 0
- joint Joint_3: limit lower=-1.6 upper=1.6 effort=200 velocity=1.0 -> lower=-1.6 upper=1.6 effort=200 velocity=0.1
- joint Joint_4: child Gripper -> Gripper_1; limit lower=-1.6 upper=1.6 effort=200 velocity=1.0 -> lower=-0.4 upper=0.4 effort=2.0 velocity=0.5
